File: hardware/Candy87.kicad_sch (KiCad schematic)
At the start: 235 parts, among them J1 ai03_ud, J2 USB_C_Receptacle_USB2.0, J3 Conn_01x07_Pin, U1 RP2040, U2 AMS1117-3.3, U3 W25Q128JVS, U4 USBLC6-2SC6, U5 74AHCT1G125, Y1 12MHz

Commit message: Minor changes
Minimal changes to USB Port:
- Removed wrong line from CC2 to A8 on USB-C
- A tiny tiny bit bigger PCB Edge around USB Port

Other:
- Added/changed Logos

New gerbers, cpl/bom stay the same (no changes)
Connections:
- net at J2.B5 (CC2), R5.2: no longer J2.A8 (SBU1)
- no-connect marks 3 -> 4
Changed lines of the file:
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@@
   (junction (at 266.7 367.03) (diameter 0) (color 0 0 0 0)
-  )
-  (junction (at 218.44 113.03) (diameter 0) (color 0 0 0 0)
   )
   (junction (at 62.23 331.47) (diameter 0) (color 0 0 0 0)
@@
   (no_connect (at 149.86 66.04))
   (no_connect (at 210.82 135.89))
+  (no_connect (at 210.82 133.35))
   (no_connect (at 386.08 85.09))
   (wire (pts (xy 219.71 255.27) (xy 219.71 285.75))
@@
     (stroke (width 0) (type default))
   )
-  (wire (pts (xy 218.44 113.03) (xy 219.71 113.03))
+  (wire (pts (xy 210.82 113.03) (xy 219.71 113.03))
     (stroke (width 0) (type default))
   )
@@
     (stroke (width 0) (type default))
   )
-  (wire (pts (xy 210.82 133.35) (xy 218.44 133.35))
-    (stroke (width 0) (type default))
-  )
   (wire (pts (xy 38.1 153.67) (xy 54.61 153.67))
     (stroke (width 0) (type default))
@@
     (stroke (width 0) (type default))
   )
-  (wire (pts (xy 210.82 113.03) (xy 218.44 113.03))
-    (stroke (width 0) (type default))
-  )
   (wire (pts (xy 24.13 255.27) (xy 24.13 270.51))
     (stroke (width 0) (type default))
@@
     (stroke (width 0) (type default))
   )
-  (wire (pts (xy 218.44 113.03) (xy 218.44 133.35))
-    (stroke (width 0) (type default))
-  )
