File: hardware/Candy87.kicad_pcb (KiCad board)
At the start: 2 copper layers, 343.6 x 123.5 mm, 254 parts, among them J1 ai03_ud, J2 USB_C_Receptacle_USB2.0, J3 Conn_01x07_Pin, U1 RP2040, U2 AMS1117-3.3, U3 W25Q128JVS, U4 USBLC6-2SC6, U5 74AHCT1G125, Y1 12MHz

Commit message: Added credits & libaries
Libaries (footprint and symbols) added in the project
Added credits and licenses for the used libaries
Updated readme with credit info
Parts:
- removed the ? at (31.3, -146.0)
- removed the ? at (40.3, -146.0)
- removed the ? at (37.9, -146.0)
- moved ? 0.22 mm to (32.4, -146.0)
- moved ? 0.15 mm to (36.9, -146.0)
- moved ? 0.13 mm to (39.4, -146.0)
